Commit message: update wheele model

File: description/collision_sensor.xacro (robot description, xacro)
@@ -1,13 +1,13 @@
 <?xml version="1.0"?>
 <robot xmlns:xacro="http://www.ros.org/wiki/xacro" >
-    <joint name="camera_joint" type="fixed">
+    <joint name="collision_joint" type="fixed">
         <parent link="chassis"/>
-        <child link="camera"/>
-        <origin xyz="${camera_x} ${camera_y} ${camera_z}" rpy="0 0 0"/>
+        <child link="collision_sensor"/>
+        <origin xyz="${collision_x} ${collision_y} ${collision_z}" rpy="${pi/2} 0 0"/>
     </joint>
-    <link name="camera">
+    <link name="collision_sensor">
         <visual>
             <geometry>
-                <box size="${camera_length} ${camera_width} ${camera_height}"/>
+                <cylinder radius="${0.02/2}" length="0.5"/>
             </geometry>
             <material name="blue"/>
@@ -15,41 +15,19 @@
         <collision>
             <geometry>
-                <box size="${camera_length} ${camera_width} ${camera_height}"/>
+                <cylinder radius="${0.02/2}" length="0.5"/>
             </geometry>
         </collision>
-        <xacro:inertial_box mass="0.5" x="${camera_length}" y="${camera_width}" z="${camera_height}">
-            <origin xyz="0 0 ${camera_height/2}" rpy="0 0 0"/>
-        </xacro:inertial_box>
+        <xacro:inertial_cylinder mass="0.1" length="0.5" radius="${0.02/2}">
+            <origin xyz="0 0 0" rpy="0 0 0"/>
+        </xacro:inertial_cylinder>
     </link>
-    <gazebo reference="camera">
-        <sensor name="Camera" type="camera">
-            <!--
-            https://en.wikipedia.org/wiki/PlayStation_Eye
-            -->
-            <pose relative_to="camera_joint">0.015 0 0 0 0 0</pose>
-            <always_on>1</always_on>
-            <update_rate>10</update_rate>
-            <topic>/gz_camera/image_raw</topic>
-            <camera>
-            <horizontal_fov>1.3</horizontal_fov>
-            <image>
-                <width>640</width>
-                <height>480</height>
-                <format>R8G8B8</format>
-            </image>
-            <clip>
-                <near>0.1</near>
-                <far>1000</far>
-            </clip>
-            <distortion>
-                <k1>-0.383727</k1>
-                <k2>0.524611</k2>
-                <p1>0.007938</p1>
-                <p2>0.033545 </p2>
-                <k3>1.991965</k3>
-                <center>0.5 0.5</center>
-            </distortion>
-            </camera>
-            <enable_metrics>true</enable_metrics>
+    <gazebo reference="collision_sensor">
+        <sensor name='sensor_contact' type='contact'>
+          <contact>
+            <collision>collision_sensor</collision>
+            <topic>/contact</topic>
+          </contact>
+          <always_on>1</always_on>
+          <update_rate>100</update_rate>
         </sensor>
     </gazebo>

File: description/lidar.xacro (robot description, xacro)
@@ -25,5 +25,5 @@
         <sensor name='LidarCircularSensor' type='gpu_lidar'>
             <pose relative_to="laser_joint">0 0 0.013 0 0 0</pose>
-            <topic>/scan</topic>
+            <topic>/scangz</topic>
             <update_rate>10</update_rate>
             <ray>
@@ -50,5 +50,5 @@
             <always_on>1</always_on>
             <visualize>true</visualize>
-            <!--<frame_id>lidar</frame_id>-->
+            <!-- <frame_id>lidar</frame_id> -->
         </sensor>
     </gazebo>

File: description/lidarAS.xacro (robot description, xacro)
@@ -25,5 +25,5 @@
         <sensor name='lidarASCircularSensor' type='gpu_lidar'>
             <pose relative_to="laserAS_joint">0.016 0.02 0.03 0 0 0</pose>
-            <topic>/lidarAS</topic>
+            <topic>/lidarASgz</topic>
             <update_rate>10</update_rate>
             <ray>

File: description/macros_gazebo_control.xacro (robot description, xacro)
@@ -20,5 +20,5 @@
             <min_acceleration>-5</min_acceleration>
             <max_acceleration>5</max_acceleration>
-            <topic>/model/base_link/cmd_vel0</topic>
+            <topic>/cmd_vel0</topic>
         </plugin>
         <plugin
@@ -40,5 +40,5 @@
             <min_acceleration>-5</min_acceleration>
             <max_acceleration>5</max_acceleration>
-            <topic>/model/base_link/cmd_vel1</topic>
+            <topic>/cmd_vel1</topic>
         </plugin>
         <plugin
@@ -61,5 +61,5 @@
             <static_update_frequency>1</static_update_frequency>
         </plugin>
-        <plugin
+        <!-- <plugin
             filename="gz-sim-odometry-publisher-system"
             name="gz::sim::systems::OdometryPublisher">
@@ -67,5 +67,5 @@
             <odom_topic>/odom</odom_topic>
             <robot_base_frame>base_link</robot_base_frame>
-        </plugin>
+        </plugin> -->
     </gazebo>
 </robot>

File: description/model.urdf.xacro (robot description, xacro)
@@ -4,4 +4,7 @@
     <xacro:include filename="macros_gazebo_control.xacro" />
     <xacro:include filename="lidar.xacro" />
+    <xacro:include filename="gps.xacro" />
+    <xacro:include filename="imu.xacro" />
+    <xacro:include filename="collision_sensor.xacro" />
     <xacro:include filename="camera.xacro" />
     <xacro:include filename="lidarAS.xacro" />

File: description/tmp.urdf (robot description, URDF)
Before this commit: robot wheele, 11 links, 10 joints
Links:
- added link cam_frame, mass 0.5; collision box size=0.03 0.1 0.065; visual box size=0.03 0.1 0.065
- added link collision_sensor, mass 0.1; collision cylinder length=0.5 radius=0.01; visual cylinder length=0.5 radius=0.01
- added link gps, mass 0.1; collision cylinder length=0.02 radius=0.01; visual cylinder length=0.02 radius=0.01
- added link imu, mass 0.001; collision box size=0.01 0.01 0.005; visual box size=0.01 0.01 0.005
- added link laser, mass 0.1; collision cylinder length=0.04 radius=0.019; visual cylinder length=0.04 radius=0.019
- added link lidarAS, mass 0.5; collision box size=0.032 0.076 0.22; visual box size=0.032 0.076 0.22
Joints:
- added joint camera_joint: type fixed, parent chassis, child cam_frame, origin xyz=0.2515 0.003500000000000003 0.1705 rpy=0 0 0
- added joint collision_joint: type fixed, parent chassis, child collision_sensor, origin xyz=0.3165 0 0.07 rpy=1.5707963267948966 0 0
- added joint gps_joint: type fixed, parent chassis, child gps, origin xyz=-0.1915 -0.1065 0.29300000000000004 rpy=0 0 0
- added joint imu_joint: type fixed, parent chassis, child imu, origin xyz=0.041499999999999995 0.0 0.203 rpy=0 0 0
- added joint laserAS_joint: type fixed, parent chassis, child lidarAS, origin xyz=-0.1405 0.11649999999999999 0.303 rpy=0 0 0
- added joint laser_joint: type fixed, parent chassis, child laser, origin xyz=0.19649999999999998 -0.1075 0.213 rpy=0 0 0
- joint base_footprint_joint: child base_footprint -> base_link; parent base_link -> base_footprint

File: description/wheele_core.xacro (robot description, xacro)
@@ -27,4 +27,10 @@
     <xacro:property name="lidar_y" value="${-chassis_width/2 + 0.03 + 0.038/2}"/>
     <xacro:property name="lidar_z" value="${chassis_height+0.02}"/>
+    <xacro:property name="gps_x" value="${-wheelbase_length/2 - 0.035}"/>
+    <xacro:property name="gps_y" value="${-chassis_width/2 + 0.05}"/>
+    <xacro:property name="gps_z" value="${chassis_height+0.10}"/>
+    <xacro:property name="imu_x" value="${wheelbase_length/2 -0.115}"/>
+    <xacro:property name="imu_y" value="${0.0}"/>
+    <xacro:property name="imu_z" value="${chassis_height+0.01}"/>
     <xacro:property name="camera_width" value="0.1"/>
     <xacro:property name="camera_height" value="0.065"/>
@@ -34,4 +40,7 @@
     <xacro:property name="camera_y" value="${-chassis_width/2 + 0.16}"/>
     <xacro:property name="camera_z" value="${0.078 + 0.06 + camera_height/2}"/>
+    <xacro:property name="collision_x" value="${wheelbase_length/2 + 0.16}"/>
+    <xacro:property name="collision_y" value="${0}"/>
+    <xacro:property name="collision_z" value="${0.07}"/>
     <xacro:property name="lidarAS_width" value="0.076"/>
     <xacro:property name="lidarAS_height" value="0.220"/>
@@ -87,13 +96,13 @@
     </xacro:macro>
     <!-- BASE LINK -->
-    <link name="base_link">
+    <link name="base_footprint">
     </link>
     <!-- BASE_FOOTPRINT LINK -->
     <joint name="base_footprint_joint" type="fixed">
+        <child link="base_footprint"/>
         <parent link="base_link"/>
-        <child link="base_footprint"/>
         <origin xyz="0 0 0" rpy="0 0 0"/>
     </joint>
-    <link name="base_footprint">
+    <link name="base_link">
     </link>
     <!-- CHASSIS LINK -->
@@ -128,5 +137,5 @@
     <xacro:wheel prefix="rear_right" reflect_x="-1" reflect_y="1" />
     <xacro:wheel prefix="rear_left" reflect_x="-1" reflect_y="-1" />
-    <!-- LEFT WHEEL LINK
+     <!-- LEFT WHEEL LINK
     <joint name="left_wheel_joint" type="continuous">
         <parent link="base_link"/>
